Commit message: Added second realsense camera at rear.

File: husky_description/urdf/accessories/intel_realsense_with_ir_stereo.urdf.xacro (robot description, xacro)
@@ -68,4 +68,68 @@
         </sensor>
       </gazebo>
+    <!-- added code for greyscale "IR" stereo camera-->
+    <!-- Stereo Camera Sensor Front Start -->
+    <!-- chage camera lens seperation distances to real values -->
+    <gazebo reference="${frame}">
+        <sensor type="multicamera" name="${prefix}_realsense_stereo">
+            <update_rate>30.0</update_rate>
+            <camera name="left">
+                <pose>0 0.02 0 0 0 0</pose> <!-- x y z r p y -->
+                <!-- 75x65 degree FOV for the depth sensor -->
+                <horizontal_fov>1.5184351666666667</horizontal_fov>
+                <vertical_fov>1.0122901111111111</vertical_fov>
+                <image>
+                    <width>848</width>
+                    <height>800</height>
+                    <format>L8</format> <!-- L8 is greysacle use R8G8B8 for color -->
+                </image>
+                <clip>
+                    <near>0.02</near>
+                    <far>300</far>
+                </clip>
+                <noise>
+                    <type>gaussian</type>
+                    <mean>0.0</mean>
+                    <stddev>0.007</stddev>
+                </noise>
+            </camera>
+            <camera name="right">
+                <pose>0 -0.02 0 0 0 0</pose> <!-- x y z r p y -->
+                <!-- 75x65 degree FOV for the depth sensor -->
+                <horizontal_fov>1.5184351666666667</horizontal_fov>
+                <vertical_fov>1.0122901111111111</vertical_fov>
+                <image>
+                    <width>848</width>
+                    <height>800</height>
+                    <format>L8</format> <!-- L8 is greysacle use R8G8B8 for color -->
+                </image>
+                <clip>
+                    <near>0.02</near>
+                    <far>300</far>
+                </clip>
+                <noise>
+                    <type>gaussian</type>
+                    <mean>0.0</mean>
+                    <stddev>0.007</stddev>
+                </noise>
+            </camera>
+            <plugin name="stereo_camera_controller" filename="libgazebo_ros_multicamera.so">
+                <alwaysOn>true</alwaysOn>
+                <updateRate>0.0</updateRate>
+                <cameraName>${topic}</cameraName>
+                <imageTopicName>image_raw</imageTopicName>
+                <cameraInfoTopicName>camera_info</cameraInfoTopicName>
+                <frameName>${frame}_gazebo</frameName>
+                <!--<rightFrameName>right_camera_optical_frame</rightFrameName>-->
+                <hackBaseline>0.07</hackBaseline>
+                <distortionK1>0.0</distortionK1>
+                <distortionK2>0.0</distortionK2>
+                <distortionK3>0.0</distortionK3>
+                <distortionT1>0.0</distortionT1>
+                <distortionT2>0.0</distortionT2>
+            </plugin>
+        </sensor>
+    </gazebo>
+    <!-- added code for greyscale "IR" stereo camera-->
     </xacro:macro>
     <link name="${prefix}_realsense_lens">
@@ -93,4 +157,5 @@
       <child link="${prefix}_realsense" />
     </joint>
+    <!-- Stereo Camera Sensor Front End -->
     <xacro:intel_realsense frame="${prefix}_realsense" topic="${topic}"/>
   </xacro:macro>

File: husky_description/urdf/husky.urdf.xacro (robot description, xacro)
@@ -47,4 +47,10 @@
   <xacro:arg name="realsense_rpy" default="$(optenv HUSKY_REALSENSE_RPY 0 0 0)" />
   <xacro:arg name="realsense_mount" default="$(optenv HUSKY_REALSENSE_MOUNT_FRAME sensor_arch_mount_link)" />
+  <!-- added code for second realsense camera -->
+  <xacro:arg name="realsense_rear_enabled" default="$(optenv HUSKY_REALSENSE_SECONDARY_ENABLED 0)" />
+  <xacro:arg name="realsense_rear_xyz" default="$(optenv HUSKY_REALSENSE_SECONDARY_XYZ 0 0 0)" />
+  <xacro:arg name="realsense_rear_rpy" default="$(optenv HUSKY_REALSENSE_SECONDARY_RPY 0 0 0)" />
+  <xacro:arg name="realsense_rear_mount" default="$(optenv HUSKY_REALSENSE_SECONDARY_MOUNT_FRAME sensor_arch_mount_link)" />
+  <!-- added code for second realsense camera -->
   <xacro:property name="husky_front_bumper_extend" value="$(optenv HUSKY_FRONT_BUMPER_EXTEND 0)" />
   <xacro:property name="husky_rear_bumper_extend" value="$(optenv HUSKY_REAR_BUMPER_EXTEND 0)" />
@@ -196,4 +202,16 @@
     <xacro:intel_realsense_mount prefix="camera" topic="realsense" parent_link="realsense_mountpoint"/>
   </xacro:if>
+  <!-- added code -->
+  <!-- add the second intel realsense to the sensor arch if needed -->
+  <xacro:if value="$(arg realsense_rear_enabled)">
+    <link name="realsense_rear_mountpoint"/>
+    <joint name="realsense_rear_mountpoint_joint" type="fixed">
+      <origin xyz="$(arg realsense_rear_xyz)" rpy="$(arg realsense_rear_rpy)" />
+      <parent link="$(arg realsense_rear_mount)"/>
+      <child link="realsense_rear_mountpoint" />
+    </joint>
+    <xacro:intel_realsense_mount prefix="camera_rear" topic="realsense_rear" parent_link="realsense_rear_mountpoint"/>
+  </xacro:if>
+  <!-- added code -->
   <!--
     Add the 3d laser to the sensor arch if needed
